Commit message: add urg

File: icart_mini_description/urdf/icart_mini.xacro (robot description, xacro)
@@ -6,4 +6,5 @@
   <xacro:property name="camera_link" value="0.05"/> <!-- Size of square 'camera' box -->
   <xacro:property name="hokuyo_link" value="0.1" /> <!-- Size of square 'hokuyo' box -->
+  <xacro:property name="hokuyo2_link" value="0.1" /> <!-- Size of square 'hokuyo' box -->
   <!-- Import all Gazebo-customization elements, including Gazebo colors -->
   <xacro:include filename="$(find icart_mini_description)/urdf/icart_mini.gazebo" />
@@ -141,9 +142,34 @@
     <child link="hokuyo_link"/>
   </joint>
-  <link name="hokuyo_link">
+    <link name="hokuyo_link">
     <collision>
       <origin xyz="0 0 0" rpy="0 0 0"/>
       <geometry>
         <box size="${hokuyo_link} ${hokuyo_link} ${hokuyo_link}"/>
+      </geometry>
+    </collision>
+    <visual>
+      <origin xyz="0 0 0" rpy="0 0 0"/>
+      <geometry>
+        <mesh filename="package://icart_mini_description/meshes/hokuyo.dae"/>
+      </geometry>
+    </visual>
+    <inertial>
+      <mass value="0.0001"/>
+      <origin xyz="0 0 0" rpy="0 0 0"/>
+      <inertia ixx="0.0001" ixy="0" ixz="0" iyy="0.0001" iyz="0" izz="0.0001"/>
+    </inertial>
+  </link>
+  <joint name="hokuyo2_joint" type="fixed">
+    <axis xyz="0 1 0"/>
+    <origin xyz="0.243 0 0.5" rpy="0 0.7 0"/>
+    <parent link="base_link"/>
+    <child link="hokuyo2_link"/>
+  </joint>
+  <link name="hokuyo2_link">
+    <collision>
+      <origin xyz="0 0 0" rpy="0 0 0"/>
+      <geometry>
+        <box size="${hokuyo2_link} ${hokuyo2_link} ${hokuyo2_link}"/>
       </geometry>
     </collision>

Commit message: fix

File: icart_mini_description/urdf/icart_mini.xacro (robot description, xacro)
@@ -6,5 +6,5 @@
   <xacro:property name="camera_link" value="0.05"/> <!-- Size of square 'camera' box -->
   <xacro:property name="hokuyo_link" value="0.1" /> <!-- Size of square 'hokuyo' box -->
-  <xacro:property name="hokuyo2_link" value="0.1" /> <!-- Size of square 'hokuyo' box -->
+  <xacro:property name="velodyne_link" value="0.1" /> <!-- Size of square 'hokuyo' box -->
   <!-- Import all Gazebo-customization elements, including Gazebo colors -->
   <xacro:include filename="$(find icart_mini_description)/urdf/icart_mini.gazebo" />
@@ -161,15 +161,15 @@
     </inertial>
   </link>
-  <joint name="hokuyo2_joint" type="fixed">
-    <axis xyz="0 1 0"/>
-    <origin xyz="0.243 0 0.5" rpy="0 0.7 0"/>
+  <joint name="velodyne_joint" type="fixed">
+    <axis xyz="0 1 0"/>
+    <origin xyz="0.243 0 0.5" rpy="0 0 0"/>
     <parent link="base_link"/>
-    <child link="hokuyo2_link"/>
-  </joint>
-  <link name="hokuyo2_link">
-    <collision>
-      <origin xyz="0 0 0" rpy="0 0 0"/>
-      <geometry>
-        <box size="${hokuyo2_link} ${hokuyo2_link} ${hokuyo2_link}"/>
+    <child link="velodyne_link"/>
+  </joint>
+  <link name="velodyne_link">
+    <collision>
+      <origin xyz="0 0 0" rpy="0 0 0"/>
+      <geometry>
+        <box size="${velodyne_link} ${velodyne_link} ${velodyne_link}"/>
       </geometry>
     </collision>

Commit message: -

File: icart_mini_description/urdf/icart_mini.xacro (robot description, xacro)
@@ -6,5 +6,5 @@
   <xacro:property name="camera_link" value="0.05"/> <!-- Size of square 'camera' box -->
   <xacro:property name="hokuyo_link" value="0.1" /> <!-- Size of square 'hokuyo' box -->
-  <xacro:property name="velodyne_link" value="0.1" /> <!-- Size of square 'hokuyo' box -->
+  <xacro:property name="velodyne_link" value="0.1" /> <!-- Size of square 'velodyne' box -->
   <!-- Import all Gazebo-customization elements, including Gazebo colors -->
   <xacro:include filename="$(find icart_mini_description)/urdf/icart_mini.gazebo" />

Commit message: fix

File: icart_mini_description/urdf/icart_mini.xacro (robot description, xacro)
@@ -6,5 +6,5 @@
   <xacro:property name="camera_link" value="0.05"/> <!-- Size of square 'camera' box -->
   <xacro:property name="hokuyo_link" value="0.1" /> <!-- Size of square 'hokuyo' box -->
-  <xacro:property name="velodyne_link" value="0.1" /> <!-- Size of square 'velodyne' box -->
+  <xacro:property name="velodyne_link" value="0.1" /> <!-- Size of square '3durg' box -->
   <!-- Import all Gazebo-customization elements, including Gazebo colors -->
   <xacro:include filename="$(find icart_mini_description)/urdf/icart_mini.gazebo" />

Commit message: -

File: icart_mini_description/urdf/icart_mini.xacro (robot description, xacro)
@@ -163,5 +163,5 @@
   <joint name="velodyne_joint" type="fixed">
     <axis xyz="0 1 0"/>
-    <origin xyz="0.243 0 0.5" rpy="0 0 0"/>
+    <origin xyz="0.243 0 0.5" rpy="0 0.4 0"/>
     <parent link="base_link"/>
     <child link="velodyne_link"/>

Commit message: -

File: icart_mini_description/urdf/icart_mini.xacro (robot description, xacro)
@@ -6,5 +6,5 @@
   <xacro:property name="camera_link" value="0.05"/> <!-- Size of square 'camera' box -->
   <xacro:property name="hokuyo_link" value="0.1" /> <!-- Size of square 'hokuyo' box -->
-  <xacro:property name="velodyne_link" value="0.1" /> <!-- Size of square '3durg' box -->
+  <xacro:property name="hokuyo3d_link" value="0.1" /> <!-- Size of square '3durg' box -->
   <!-- Import all Gazebo-customization elements, including Gazebo colors -->
   <xacro:include filename="$(find icart_mini_description)/urdf/icart_mini.gazebo" />
@@ -142,5 +142,5 @@
     <child link="hokuyo_link"/>
   </joint>
-    <link name="hokuyo_link">
+  <link name="hokuyo_link">
     <collision>
       <origin xyz="0 0 0" rpy="0 0 0"/>
@@ -161,15 +161,15 @@
     </inertial>
   </link>
-  <joint name="velodyne_joint" type="fixed">
-    <axis xyz="0 1 0"/>
-    <origin xyz="0.243 0 0.5" rpy="0 0.4 0"/>
+  <joint name="hokuyo3d_joint" type="fixed">
+    <axis xyz="0 1 0"/>
+    <origin xyz="0.27 0 0.35" rpy="0 0.034 0"/>
     <parent link="base_link"/>
-    <child link="velodyne_link"/>
-  </joint>
-  <link name="velodyne_link">
-    <collision>
-      <origin xyz="0 0 0" rpy="0 0 0"/>
-      <geometry>
-        <box size="${velodyne_link} ${velodyne_link} ${velodyne_link}"/>
+    <child link="hokuyo3d_link"/>
+  </joint>
+  <link name="hokuyo3d_link">
+    <collision>
+      <origin xyz="0 0 0" rpy="0 0 0"/>
+      <geometry>
+        <box size="${hokuyo3d_link} ${hokuyo3d_link} ${hokuyo3d_link}"/>
       </geometry>
     </collision>

Commit message: include imu.urdf into icart_mini.xacro

File: icart_mini_description/urdf/icart_mini.xacro (robot description, xacro)
@@ -6,14 +6,12 @@
   <xacro:property name="camera_link" value="0.05"/> <!-- Size of square 'camera' box -->
   <xacro:property name="hokuyo_link" value="0.1" /> <!-- Size of square 'hokuyo' box -->
-  <!-- Import all Gazebo-customization elements, including Gazebo colors -->
-  <xacro:include filename="$(find icart_mini_description)/urdf/icart_mini.gazebo" />
   <!-- Import Rviz colors -->
   <xacro:include filename="$(find icart_mini_description)/urdf/materials.xacro" />
   <!-- Used for fixing robot to Gazebo 'base_link' -->
-  <!--link name="world"/>
+  <link name="world"/>
   <joint name="continuous" type="continuous">
     <parent link="world"/>
     <child link="base_link"/>
-  </joint-->
+  </joint>
   <!-- Base Link -->
   <link name="base_link">
@@ -206,3 +204,9 @@
     </actuator>
   </transmission>
+  <!-- Import all Gazebo-customization elements, including Gazebo colors -->
+  <xacro:include filename="$(find icart_mini_description)/urdf/icart_mini.gazebo"/>
+  <xacro:include filename="$(find icart_mini_description)/urdf/sensors/imu.urdf.xacro"/>
+  <xacro:sensor_imu name="imu" parent="base_link">
+      <origin xyz="-0.18 0.0 0.170" rpy="0 0 0"/>
+  </xacro:sensor_imu>
 </robot>

Commit message: modified to not include gazebo plugins

File: icart_mini_description/urdf/icart_mini.xacro (robot description, xacro)
@@ -204,9 +204,3 @@
     </actuator>
   </transmission>
-  <!-- Import all Gazebo-customization elements, including Gazebo colors -->
-  <xacro:include filename="$(find icart_mini_description)/urdf/icart_mini.gazebo"/>
-  <xacro:include filename="$(find icart_mini_description)/urdf/sensors/imu.urdf.xacro"/>
-  <xacro:sensor_imu name="imu" parent="base_link">
-      <origin xyz="-0.18 0.0 0.170" rpy="0 0 0"/>
-  </xacro:sensor_imu>
 </robot>

Commit message: delete camera_link

File: icart_mini_description/urdf/icart_mini.xacro (robot description, xacro)
@@ -4,5 +4,4 @@
   <!-- Constants for robot dimensions -->
   <xacro:property name="PI" value="3.1415926535897931"/>
-  <xacro:property name="camera_link" value="0.05"/> <!-- Size of square 'camera' box -->
   <xacro:property name="hokuyo_link" value="0.1" /> <!-- Size of square 'hokuyo' box -->
   <!-- Import Rviz colors -->
@@ -158,30 +157,4 @@
     </inertial>
   </link>
-  <joint name="camera_joint" type="fixed">
-    <axis xyz="0 1 0" />
-    <origin xyz="0 0 0.2" rpy="0 0 0"/>
-    <parent link="base_link"/>
-    <child link="camera_link"/>
-  </joint>
-  <link name="camera_link">
-    <collision>
-      <origin xyz="0 0 0" rpy="0 0 0"/>
-      <geometry>
-        <box size="${camera_link} ${camera_link} ${camera_link}"/>
-      </geometry>
-    </collision>
-    <visual>
-      <origin xyz="0 0 0" rpy="0 0 0"/>
-      <geometry>
-        <box size="${camera_link} ${camera_link} ${camera_link}"/>
-      </geometry>
-      <material name="red"/>
-    </visual>
-    <inertial>
-      <mass value="0.0001"/>
-      <origin xyz="0 0 0" rpy="0 0 0"/>
-      <inertia ixx="0.0001" ixy="0" ixz="0" iyy="0.0001" iyz="0" izz="0.0001"/>
-    </inertial>
-  </link>
   <transmission name="tran1">
     <type>transmission_interface/SimpleTransmission</type>

Commit message: fix the problem that robot can't move on the gazebo

File: icart_mini_description/urdf/icart_mini.xacro (robot description, xacro)
@@ -7,10 +7,5 @@
   <!-- Import Rviz colors -->
   <xacro:include filename="$(find icart_mini_description)/urdf/materials.xacro" />
-  <!-- Used for fixing robot to Gazebo 'base_link' -->
-  <link name="world"/>
-  <joint name="continuous" type="continuous">
-    <parent link="world"/>
-    <child link="base_link"/>
-  </joint>
+  <xacro:include filename="$(find icart_mini_description)/urdf/icart_mini.gazebo"/>
   <!-- Base Link -->
   <link name="base_link">

Commit message: part sensor_hokuyo frame

File: icart_mini_description/urdf/icart_mini.xacro (robot description, xacro)
@@ -4,5 +4,4 @@
   <!-- Constants for robot dimensions -->
   <xacro:property name="PI" value="3.1415926535897931"/>
-  <xacro:property name="hokuyo_link" value="0.1" /> <!-- Size of square 'hokuyo' box -->
   <!-- Import Rviz colors -->
   <xacro:include filename="$(find icart_mini_description)/urdf/materials.xacro" />
@@ -127,29 +126,4 @@
     <limit effort="100" velocity="100.0"  lower="-5000" upper="5000" />
   </joint>
-  <joint name="hokuyo_joint" type="fixed">
-    <axis xyz="0 1 0"/>
-    <origin xyz="0.243 0 0.2" rpy="0 0 0"/>
-    <parent link="base_link"/>
-    <child link="hokuyo_link"/>
-  </joint>
-  <link name="hokuyo_link">
-    <collision>
-      <origin xyz="0 0 0" rpy="0 0 0"/>
-      <geometry>
-        <box size="${hokuyo_link} ${hokuyo_link} ${hokuyo_link}"/>
-      </geometry>
-    </collision>
-    <visual>
-      <origin xyz="0 0 0" rpy="0 0 0"/>
-      <geometry>
-        <mesh filename="package://icart_mini_description/meshes/hokuyo.dae"/>
-      </geometry>
-    </visual>
-    <inertial>
-      <mass value="0.0001"/>
-      <origin xyz="0 0 0" rpy="0 0 0"/>
-      <inertia ixx="0.0001" ixy="0" ixz="0" iyy="0.0001" iyz="0" izz="0.0001"/>
-    </inertial>
-  </link>
   <transmission name="tran1">
     <type>transmission_interface/SimpleTransmission</type>

Commit message: fix icart_mini.xacor

File: icart_mini_description/urdf/icart_mini.xacro (robot description, xacro)
@@ -10,18 +10,18 @@
   <link name="base_link">
     <collision>
-      <origin xyz="0 0 0.1" rpy="0 0 0"/>
+      <origin xyz="-0.15 0 0.1" rpy="0 0 0"/>
       <geometry>
-	<box size=".485 .43 .15"/>
+	    <box size=".485 .43 .15"/>
       </geometry>
     </collision>
     <visual>
-      <origin xyz="0 0 0.1" rpy="0 0 0"/>
+      <origin xyz="-0.15 0 0.1" rpy="0 0 0"/>
       <geometry>
-	<box size=".485 .43 .15"/>
+	    <box size=".485 .43 .15"/>
       </geometry>
       <material name="orange"/>
     </visual>
     <collision name="collision">
-      <origin xyz="-0.175 0.0 0.05" rpy="0 1.5707 1.5707"/>
+      <origin xyz="-0.325 0.0 0.05" rpy="0 1.5707 1.5707"/>
       <geometry>
         <cylinder  length="0.03" radius="0.04625"/>
@@ -29,22 +29,22 @@
     </collision>
     <visual name="visual">
-      <origin xyz="-0.175 0.0 0.05" rpy="0 1.5707 1.5707"/>
+      <origin xyz="-0.325 0.0 0.05" rpy="0 1.5707 1.5707"/>
       <geometry>
         <cylinder  length="0.03" radius="0.04625"/>
       </geometry>
     </visual>
-    <collision name="collision">
+    <!--collision name="collision">
       <origin xyz="0.175 0.0 0.05" rpy="0 1.5707 1.5707"/>
       <geometry>
         <cylinder  length="0.03" radius="0.04625"/>
       </geometry>
-    </collision>
+    </collision-->
     <inertial>
        <mass value="20" />
-       <origin xyz="0 0 0" rpy="0 0 0"/>
+       <origin xyz="-0.08 0 0" rpy="0 0 0"/>
        <inertia ixx="1" ixy="0" ixz="0" iyy="1" iyz="0" izz="1" />
     </inertial>
   </link>
-  <link name="visual_left_wheel">
+  <!--link name="visual_left_wheel">
     <visual name="visual">
       <origin xyz="0 0.0 0" rpy="0 1.5707 1.5707"/>
@@ -59,5 +59,5 @@
     <parent link="base_link">base_link</parent>
     <axis xyz="0 1 0"/>
-  </joint>
+  </joint-->
   <link name="left_wheel">
     <collision name="collision">
@@ -67,10 +67,10 @@
       </geometry>
     </collision>
-    <!--visual name="visual">
+    <visual name="visual">
       <origin xyz="0 0.0 0" rpy="0 1.5707 1.5707"/>
       <geometry>
         <cylinder  length="0.03" radius="0.0725"/>
       </geometry>
-    </visual-->
+    </visual>
     <inertial>
       <mass value="1" />
@@ -86,5 +86,5 @@
     <limit effort="100" velocity="100.0"  lower="-5000" upper="5000" />
   </joint>
-  <link name="visual_right_wheel">
+  <!--link name="visual_right_wheel">
     <visual name="visual">
       <origin xyz="0 0.0 0" rpy="0 1.5707 1.5707"/>
@@ -99,5 +99,5 @@
     <parent link="base_link">base_link</parent>
     <axis xyz="0 1 0"/>
-  </joint>
+  </joint-->
   <link name="right_wheel">
     <collision name="collision">
@@ -107,10 +107,10 @@
       </geometry>
     </collision>
-    <!--visual name="visual">
+    <visual name="visual">
       <origin xyz="0 0.0 0" rpy="0 1.5707 1.5707"/>
       <geometry>
         <cylinder  length="0.03" radius="0.0725"/>
       </geometry>
-    </visual-->
+    </visual>
     <inertial>
       <mass value="1" />
@@ -131,5 +131,5 @@
       <hardwareInterface>VelocityJointInterface</hardwareInterface>
     </joint>
-  <actuator name="left_motor">
+    <actuator name="left_motor">
       <hardwareInterface>VelocityJointInterface</hardwareInterface>
       <mechanicalReduction>1</mechanicalReduction>
@@ -141,5 +141,5 @@
       <hardwareInterface>VelocityJointInterface</hardwareInterface>
     </joint>
-  <actuator name="right_motor">
+    <actuator name="right_motor">
       <hardwareInterface>VelocityJointInterface</hardwareInterface>
       <mechanicalReduction>1</mechanicalReduction>
