Commit message: the imu size defined

File: icart_mini_description/urdf/sensors/imu.urdf.xacro (robot description, xacro)
@@ -3,5 +3,5 @@
                          xmlns:controller="http://playerstage.sourceforge.net/gazebo/xmlschema/#controller"
                          xmlns:interface="http://playerstage.sourceforge.net/gazebo/xmlschema/#interface">
-  <xacro:macro name="sensor_imu" params="name parent *origin">
+  <xacro:macro name="sensor_imu" params="name parent *origin size">
 	  <joint name="${name}_joint" type="fixed">
 	      <axis xyz="1 0 0"/>
@@ -20,5 +20,5 @@
 	        <origin rpy="0 0 0" xyz="0 0 0"/>
 	        <geometry>
-	          <box size="0.001 0.001 0.001"/>
+	          <box size="${size}"/>
 	        </geometry>
 	      </visual>
@@ -26,5 +26,5 @@
 	        <origin rpy="0 0 0" xyz="0 0 0"/>
 	        <geometry>
-	          <box size=".001 .001 .001"/>
+	          <box size="${size}"/>
 	        </geometry>
 	      </collision>
