Commit message: hokuyo3dノード側のframe_idがhokuyo3dのためhokuyo3dのリンクを{name}_linkから{name}に変更

File: icart_mini_description/urdf/sensors/hokuyo3d.urdf.xacro (robot description, xacro)
@@ -8,7 +8,7 @@
 	      <insert_block name="origin"/>
 	      <parent link="${parent}"/>
-	      <child link="${name}_link"/>
+	      <child link="${name}"/>
 	  </joint>
-	  <link name="${name}_link">
+	  <link name="${name}">
 	      <inertial>
 	        <mass value="0.001"/>
@@ -29,5 +29,5 @@
 	      </collision>
 	  </link>
-      <gazebo reference="${name}_link">
+      <gazebo reference="${name}">
         <sensor name="velodyne" type="ray">
         <always_on>true</always_on>
@@ -59,5 +59,5 @@
           <updateRate>20</updateRate>
           <topicName>/${name}/hokuyo_cloud</topicName>
-          <frameName>${name}_link</frameName>
+          <frameName>${name}</frameName>
         </plugin>
       </sensor>
